File: smart-outlet-t-reverse.kicad_pcb (KiCad board)
At the start: 2 copper layers, 51.3 x 32.4 mm, 33 parts, among them J1 Conn_01x01, J2 Conn_01x01, P1 Conn_01x01, P2 Conn_01x01, Q2 MMBT3904, SW1 Relay_SPST-NO, U1 BP2525

Commit message: Updated README to be more detailed. Updated schematic to pass checks and regenerated PDF. Added a few comments. Updated pcb from schematic changes.
Parts:
- C170: value 470µF -> 470µ
- C172: value 2.2µF -> 2.2µ
- C173: value 1µF -> 1µ
- C3, EC2: value 10µF -> 10µ
- R125, R20: value 510Ω -> 510
- R127: value 10kΩ -> 10k
- R148: value 3.6kΩ -> 3.6k
- R17, R18, R7, R8: value 1.3Ω -> 1.3
Connections:
- net Net-(D3-K) renamed /power supply/U1_GND
Changed lines of the file:
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@@
 	(net 3 "Net-(D2-K)")
 	(net 4 "Net-(D11-K)")
-	(net 5 "Net-(D3-K)")
+	(net 5 "/power supply/U1_GND")
 	(net 6 "Net-(Q2-B)")
 	(net 7 "FUSED_AC")
@@
 			)
 		)
-		(property "Value" "2.2µF"
+		(property "Value" "2.2µ"
 			(at 1.25 1.6 90)
 			(layer "F.Fab")
@@
 			)
 		)
-		(property "Value" "510Ω"
+		(property "Value" "510"
 			(at 0 1.43 0)
 			(layer "F.Fab")
@@
 			)
 		)
-		(property "Value" "470µF"
+		(property "Value" "470µ"
 			(at 1.25 4.4 90)
 			(layer "F.Fab")
@@
 			)
 		)
-		(property "Value" "510Ω"
+		(property "Value" "510"
 			(at 0 1.53 0)
 			(layer "F.Fab")
@@
 			)
 		)
-		(property "Value" "3.6kΩ"
+		(property "Value" "3.6k"
 			(at 0 1.65 0)
 			(layer "F.Fab")
@@
 			(layers "*.Cu" "*.Mask")
 			(remove_unused_layers no)
-			(net 5 "Net-(D3-K)")
+			(net 5 "/power supply/U1_GND")
 			(pinfunction "1")
 			(pintype "passive")
@@
 			)
 		)
-		(property "Value" "10µF"
+		(property "Value" "10µ"
 			(at 0 1.43 0)
 			(layer "F.Fab")
@@
 			)
 		)
-		(property "Value" "10µF"
+		(property "Value" "10µ"
 			(at 1.75 1.55 90)
 			(layer "F.Fab")
@@
 			)
 		)
-		(property "Value" "10kΩ"
+		(property "Value" "10k"
 			(at 3.4 0.03 90)
 			(layer "F.Fab")
@@
 			)
 		)
-		(property "Value" "1µF"
+		(property "Value" "1µ"
 			(at 0 -1.68 0)
 			(layer "B.Fab")
@@
 			(layers "B.Cu" "B.Mask" "B.Paste")
 			(roundrect_rratio 0.25)
-			(net 5 "Net-(D3-K)")
+			(net 5 "/power supply/U1_GND")
 			(pintype "passive")
 		)
@@
 			)
 		)
-		(property "Value" "1.3Ω"
+		(property "Value" "1.3"
 			(at 3.394113 -0.015787 45)
 			(layer "B.Fab")
@@
 			(layers "B.Cu" "B.Mask" "B.Paste")
 			(roundrect_rratio 0.25)
-			(net 5 "Net-(D3-K)")
+			(net 5 "/power supply/U1_GND")
 			(pintype "passive")
 		)
@@
 			)
 		)
-		(property "Value" "1.3Ω"
+		(property "Value" "1.3"
 			(at 3.323402 0.196345 45)
 			(layer "B.Fab")
@@
 			(layers "B.Cu" "B.Mask" "B.Paste")
 			(roundrect_rratio 0.25)
-			(net 5 "Net-(D3-K)")
+			(net 5 "/power supply/U1_GND")
 			(pintype "passive")
 		)
@@
 			)
 		)
-		(property "Value" "1.3Ω"
+		(property "Value" "1.3"
 			(at 3.323402 -0.227919 45)
 			(layer "B.Fab")
@@
 			(layers "B.Cu" "B.Mask" "B.Paste")
 			(roundrect_rratio 0.25)
-			(net 5 "Net-(D3-K)")
+			(net 5 "/power supply/U1_GND")
 			(pintype "passive")
 		)
@@
 			(layers "B.Cu" "B.Mask" "B.Paste")
 			(roundrect_rratio 0.15)
-			(net 5 "Net-(D3-K)")
+			(net 5 "/power supply/U1_GND")
 			(pinfunction "GND")
 			(pintype "passive")
@@
 			(layers "B.Cu" "B.Mask" "B.Paste")
 			(roundrect_rratio 0.15)
-			(net 5 "Net-(D3-K)")
+			(net 5 "/power supply/U1_GND")
 			(pinfunction "SEL")
 			(pintype "input")
@@
 			)
 		)
-		(property "Value" "1.3Ω"
+		(property "Value" "1.3"
 			(at 3.464823 0.054924 45)
 			(layer "B.Fab")
@@
 			(layers "B.Cu" "B.Mask" "B.Paste")
 			(roundrect_rratio 0.25)
-			(net 5 "Net-(D3-K)")
+			(net 5 "/power supply/U1_GND")
 			(pintype "passive")
 		)
@@
 			)
 		)
-		(property "Datasheet" "~"
+		(property "Datasheet" "https://mm.digikey.com/Volume0/opasdata/d220001/medias/docus/6778/5399_E1J%20SOD-123FL.PDF"
 			(at 0 0 90)
 			(unlocked yes)
@@
 			(layers "B.Cu" "B.Mask" "B.Paste")
 			(roundrect_rratio 0.2272727273)
-			(net 5 "Net-(D3-K)")
+			(net 5 "/power supply/U1_GND")
 			(pinfunction "K")
 			(pintype "passive")
